File: ScartPCB.kicad_sch (KiCad schematic)
At the start: 55 parts, among them J1 Conn_02x10_Odd_Even, Q1 BC847W, Q2 BC857W, U1 TPS61040DBVR

Commit message: Change it to work more like I want it to
Parts:
- removed C1: 4.7uF, Capacitor_SMD:C_0402_1005Metric, symbol Device:C
- removed C2: 10pF, Capacitor_SMD:C_0402_1005Metric, symbol Device:C
- removed C3: 1uF, Capacitor_SMD:C_0402_1005Metric, symbol Device:C
- removed C4: 100nF, Capacitor_SMD:C_0402_1005Metric, symbol Device:C
- removed CB1, CB2, CC1, CC2, CG1, CG2, CR1, CR2: 100uF, Capacitor_SMD:C_1206_3216Metric, symbol Device:C
- removed CB3, CC3, CG3, CR3: 22uF, Capacitor_SMD:C_0603_1608Metric, symbol Device:C
- removed D1, D2: D_Schottky, Diode_SMD:D_0402_1005Metric, symbol Device:D_Schottky
- removed L1: 10uH, Inductor_SMD:L_0603_1608Metric, symbol Device:L
- removed Q1: BC847W, Package_TO_SOT_SMD:SOT-323_SC-70, symbol Transistor_BJT:BC847W
- removed Q2: BC857W, Package_TO_SOT_SMD:SOT-323_SC-70, symbol Transistor_BJT:BC857W
- removed R1: 1.6M, Resistor_SMD:R_0402_1005Metric, symbol Device:R
- removed R2: 200K, Resistor_SMD:R_0402_1005Metric, symbol Device:R
- removed R3: 1K, Resistor_SMD:R_0402_1005Metric, symbol Device:R
- removed R5, R6: 1M, Resistor_SMD:R_0402_1005Metric, symbol Device:R
- removed U1: TPS61040DBVR, Footprints:TPS61040DBVR, symbol TPS61040DBVR:TPS61040DBVR
- added CB1, CG1, CR1: C_Polarized, Capacitor_Tantalum_SMD:CP_EIA-3528-21_Kemet-B_HandSolder, symbol Device:C_Polarized
- added CC1: 220uF, Capacitor_Tantalum_SMD:CP_EIA-3528-21_Kemet-B_HandSolder, symbol Device:C_Polarized
- added U1: 74LVC1G17, Package_TO_SOT_SMD:SC-74A-5_1.55x2.9mm_P0.95mm, symbol 74xGxx:74LVC1G17
- C0: footprint Capacitor_SMD:C_0402_1005Metric -> Capacitor_SMD:C_0805_2012Metric_Pad1.18x1.45mm_HandSolder
- R7, R9, RB1, RG1, RR1: footprint Resistor_SMD:R_0402_1005Metric -> Resistor_SMD:R_0805_2012Metric_Pad1.20x1.40mm_HandSolder
- R8, RC2, RG2, RR2: footprint Resistor_SMD:R_0402_1005Metric -> Resistor_SMD:R_0805_2012Metric_Pad1.20x1.40mm_HandSolder; now in the parts list
- RB2: footprint Resistor_SMD:R_0402_1005Metric -> Resistor_SMD:R_0805_2012Metric_Pad1.20x1.40mm_HandSolder; Manufacturer_Part_Number 0402WGF750JTCE -> (none); Package 0402 -> (none); now in the parts list
- RC1: value 300 -> 470; footprint Resistor_SMD:R_0402_1005Metric -> Resistor_SMD:R_0805_2012Metric_Pad1.20x1.40mm_HandSolder
Connections:
- net +5V: now also U1.5 (VCC)
- net BLUE: now also CB1.2
- net C: now also U1.2
- net C_SYNC: now also U1.4
- net GND: now also J1.13 (Pin_13), J1.14 (Pin_14), J1.4 (Pin_4), J1.5 (Pin_5), J1.9 (Pin_9), U1.3 (GND)
- net GREEN: now also CG1.2
- net RED: now also CR1.2
- net at RG1.2: now also CG1.1
- net at RB1.2: now also CB1.1
- net at RC1.2: now also CC1.2
- net at R7.1, R8.1: now also CC1.1
- net at RR1.2: now also CR1.1
- net SWITCH: no longer names the net of J1.8 (Pin_8)
- no-connect marks 10 -> 6
Other:
- note removed: "10-11V"
- note removed: "Boost converter"
- note removed: "R3 is for current limiting, just in case. It can be replaced with a 0 ohm resistor."
- company: screwbreaker -> dottedquad
- title: ScartPCB -> EasyScartPCB

Commit message: Get ready for first run
Parts:
- added JI13: Conn_01x01, Footprints:PAD1.5x1.5, symbol Connector_Generic:Conn_01x01
- C0: Manufacturer YAEGO -> (none); Manufacturer_Part_Number CC0402KRX7R7BB104 -> (none); Package 0402 -> 0805
- CB1, CG1, CR1: value C_Polarized -> 220uF
- R7, RB1, RG1, RG2, RR1, RR2: Manufacturer Royalohm -> (none); Manufacturer_Part_Number 0402WGF750JTCE -> (none); Package 0402 -> 0805
- R8, RC1, RC2: Package 0402 -> 0805
- R9: Manufacturer Royalohm -> (none); Manufacturer_Part_Number HP02WAF1800TCE -> (none); Package 0402 -> 0805
- RB2: Manufacturer Royalohm -> (none); Package (none) -> 0805
Connections:
- net GND: now also JI13.1 (Pin_1)
Other:
- note added: "Decoupling"
- note removed: "Descoupling"
- moved on the sheet: CB1, CC1, CG1, CR1, JP1, JP2, JP3, R7, R8, R9, RB1, RB2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
